File: Project/Backbird 002 Slimline PCB.sch (KiCad schematic (older format))
At the start: 12 parts

Commit message: Removed extra connectors from PCB
Parts:
- removed Power_4pin1: Conn_01x04, ProjectFootprints:MOLEX_8981_Generic, symbol Backbird-002-Slimline-PCB-rescue:Conn_01x04
- removed Sata_Data2: Conn_01x07, ProjectFootprints:SATA_DATA_678007005_CustomPad, symbol Backbird-002-Slimline-PCB-rescue:Conn_01x07
- +5V_Hole1, GND_Hole2: footprint Wire_Pads:SolderWirePad_single_1-2mmDrill -> Wire_Pads:SolderWirePad_single_0-8mmDrill
Changed lines of the file:
@@
-$EndComp
-$Comp
-L Backbird-002-Slimline-PCB-rescue:Conn_01x07 Sata_Data2
-U 1 1 5B19E3C5
-P 3650 4750
-F 0 "Sata_Data2" H 3570 5267 50  0000 C CNN
-F 1 "Conn_01x07" H 3570 5176 50  0000 C CNN
-F 2 "ProjectFootprints:SATA_DATA_678007005_CustomPad" H 3650 4750 50  0001 C CNN
-F 3 "" H 3650 4750 50  0001 C CNN
-	1    3650 4750
-	-1   0    0    -1
-$EndComp
-Text GLabel 3850 4450 2    60   Input ~ 0
-GND
-Text GLabel 3850 4750 2    60   Input ~ 0
-GND
-Text GLabel 3850 4550 2    60   Input ~ 0
-A+
-Text GLabel 3850 4650 2    60   Input ~ 0
-A-
-Text GLabel 3850 4850 2    60   Input ~ 0
-B-
-Text GLabel 3850 4950 2    60   Input ~ 0
-B+
-Text GLabel 3850 5050 2    60   Input ~ 0
-GND
-$Comp
-L Backbird-002-Slimline-PCB-rescue:Conn_01x04 Power_4pin1
-U 1 1 5B1AF5DD
-P 4550 5450
-F 0 "Power_4pin1" H 4550 5650 50  0000 C CNN
-F 1 "Conn_01x04" H 4550 5150 50  0000 C CNN
-F 2 "ProjectFootprints:MOLEX_8981_Generic" H 4550 5450 50  0001 C CNN
-F 3 "" H 4550 5450 50  0001 C CNN
-	1    4550 5450
-	1    0    0    -1
 $EndComp
 $Comp
@@
 F 0 "+5V_Hole1" H 3750 2000 50  0000 R CNN
 F 1 "Conn_01x01" H 3800 2100 50  0000 R CNN
-F 2 "Wire_Pads:SolderWirePad_single_1-2mmDrill" H 3200 2050 50  0001 C CNN
+F 2 "Wire_Pads:SolderWirePad_single_0-8mmDrill" H 3200 2050 50  0001 C CNN
 F 3 "~" H 3200 2050 50  0001 C CNN
 	1    3200 2050
@@
 F 0 "GND_Hole2" H 4280 2092 50  0000 L CNN
 F 1 "Conn_01x01" H 4280 2001 50  0000 L CNN
-F 2 "Wire_Pads:SolderWirePad_single_1-2mmDrill" H 4200 2050 50  0001 C CNN
+F 2 "Wire_Pads:SolderWirePad_single_0-8mmDrill" H 4200 2050 50  0001 C CNN
 F 3 "~" H 4200 2050 50  0001 C CNN
 	1    4200 2050
@@
 Text GLabel 3550 3050 0    60   Input ~ 0
 GND
-Text GLabel 4350 5650 0    60   Input ~ 0
-+5V
-Text GLabel 4350 5550 0    60   Input ~ 0
-GND
-Text GLabel 4350 5450 0    60   Input ~ 0
-GND
-Text GLabel 4350 5350 0    60   Input ~ 0
-+12V
 $Comp
 L Connector:Conn_01x01 Screw_Hole_B1

Commit message: Moved silk screen of resistors and LED power holes to be on the PCB.
Parts:
- Screw_Hole_T1: footprint ProjectFootprints:Blackbird002_Slimline_PCB_Screw -> ProjectFootprints:Blackbird002_Slimline_PCB_Screw_Long
Changed lines of the file:
@@
 F 0 "Screw_Hole_T1" H 2579 1392 50  0000 L CNN
 F 1 "Conn_01x01" H 2579 1301 50  0000 L CNN
-F 2 "ProjectFootprints:Blackbird002_Slimline_PCB_Screw" H 2500 1350 50  0001 C CNN
+F 2 "ProjectFootprints:Blackbird002_Slimline_PCB_Screw_Long" H 2500 1350 50  0001 C CNN
 F 3 "~" H 2500 1350 50  0001 C CNN
 	1    2500 1350
