File: Project/Backbird 002 Slimline PCB.sch (KiCad schematic (older format))
At the start: 10 parts

Commit message: remove extra 2 holes for the LED section
Parts:
- removed +5V_Hole1, GND_Hole2: Conn_01x01, Wire_Pads:SolderWirePad_single_0-8mmDrill, symbol Connector:Conn_01x01
Connections:
- net labels removed: +12V
- no-connect marks 4 -> 5
Changed lines of the file:
@@
-	1    0    0    -1
-$EndComp
-$Comp
-L Connector:Conn_01x01 +5V_Hole1
-U 1 1 5B1B7221
-P 3200 2050
-F 0 "+5V_Hole1" H 3750 2000 50  0000 R CNN
-F 1 "Conn_01x01" H 3800 2100 50  0000 R CNN
-F 2 "Wire_Pads:SolderWirePad_single_0-8mmDrill" H 3200 2050 50  0001 C CNN
-F 3 "~" H 3200 2050 50  0001 C CNN
-	1    3200 2050
-	-1   0    0    1
-$EndComp
-$Comp
-L Connector:Conn_01x01 GND_Hole2
-U 1 1 5B1B7286
-P 4200 2050
-F 0 "GND_Hole2" H 4280 2092 50  0000 L CNN
-F 1 "Conn_01x01" H 4280 2001 50  0000 L CNN
-F 2 "Wire_Pads:SolderWirePad_single_0-8mmDrill" H 4200 2050 50  0001 C CNN
-F 3 "~" H 4200 2050 50  0001 C CNN
-	1    4200 2050
 	1    0    0    -1
 $EndComp
@@
 Text GLabel 2750 5450 0    60   Input ~ 0
 GND
-Text GLabel 2750 5350 0    60   Input ~ 0
-+12V
 Text GLabel 3400 2050 3    60   Input ~ 0
 +5V
@@
 $EndComp
 NoConn ~ 2300 1350
+NoConn ~ 2750 5350
 $EndSCHEMATC
